Commit message: working urdf file

File: src/lane_following/urdf/lane_robot.urdf.xacro (robot description, xacro)
@@ -1,4 +1,10 @@
 <?xml version="1.0"?>
 <robot name="lane_robot" xmlns:xacro="http://ros.org/wiki/xacro">
+  <material name="blue">
+    <color rgba="0 0 1 1"/>
+  </material>
+  <material name="black">
+    <color rgba="0 0 0 1"/>
+  </material>
   <link name="base_link">
     <visual>
@@ -6,12 +12,77 @@
         <box size="0.3 0.2 0.1"/>
       </geometry>
+      <origin xyz="0 0 0.05"/>
       <material name="blue"/>
     </visual>
+    <collision>
+      <geometry>
+        <box size="0.3 0.2 0.1"/>
+      </geometry>
+      <origin xyz="0 0 0.05"/>
+    </collision>
+    <inertial>
+      <mass value="1.0"/>
+      <inertia ixx="0.01" ixy="0.0" ixz="0.0"
+               iyy="0.01" iyz="0.0"
+               izz="0.02"/>
+    </inertial>
   </link>
   <!-- Wheels -->
-  <link name="left_wheel"/>
-  <link name="right_wheel"/>
+  <link name="left_wheel">
+    <visual>
+      <geometry>
+        <cylinder length="0.05" radius="0.05"/>  <!-- 5cm radius, 5cm thick -->
+      </geometry>
+      <origin rpy="1.5707 0 0" xyz="0 0 0"/>
+      <material name="black"/>
+    </visual>
+    <collision>
+      <geometry>
+        <cylinder length="0.05" radius="0.05"/>
+      </geometry>
+       <origin rpy="1.5707 0 0" xyz="0 0 0"/>
+    </collision>
+    <inertial>
+      <mass value="0.2"/>
+      <inertia ixx="0.001" iyy="0.001" izz="0.001"
+               ixy="0.0" ixz="0.0" iyz="0.0"/>
+    </inertial>
+  </link>
+  <link name="right_wheel">
+    <visual>
+      <geometry>
+        <cylinder length="0.05" radius="0.05"/>
+      </geometry>
+      <origin rpy="1.5707 0 0" xyz="0 0 0"/>
+      <material name="black"/>
+    </visual>
+    <collision>
+      <geometry>
+        <cylinder length="0.05" radius="0.05"/>
+      </geometry>
+       <origin rpy="1.5707 0 0" xyz="0 0 0"/>
+    </collision>
+    <inertial>
+      <mass value="0.2"/>
+      <inertia ixx="0.001" iyy="0.001" izz="0.001"
+               ixy="0.0" ixz="0.0" iyz="0.0"/>
+    </inertial>
+  </link>
+  <!-- Joint: left wheel to base -->
+  <joint name="left_wheel_joint" type="continuous">
+    <parent link="base_link"/>
+    <child link="left_wheel"/>
+    <origin xyz="0 0.1 0.05" rpy="0 0 0"/>
+    <axis xyz="0 1 0"/>
+  </joint>
+  <!-- Joint: right wheel to base -->
+  <joint name="right_wheel_joint" type="continuous">
+    <parent link="base_link"/>
+    <child link="right_wheel"/>
+    <origin xyz="0 -0.1 0.05" rpy="0 0 0"/>
+    <axis xyz="0 1 0"/>
+  </joint>
   <!-- Differential Drive Plugin -->
-  <gazebo>
+  <!-- <gazebo>
     <plugin name="diff_drive" filename="libgazebo_ros_diff_drive.so">
       <ros>
@@ -23,8 +94,22 @@
       <odometry_topic>odom</odometry_topic>
     </plugin>
-  </gazebo>
-  <!-- Camera -->
+  </gazebo> -->
+  <!-- Camera sensor -->
   <link name="camera_link">
-    <sensor type="camera" name="camera_sensor">
+    <visual>
+      <geometry>
+        <box size="0.05 0.05 0.05"/>
+      </geometry>
+      <origin xyz="0 0 0"/>
+    </visual>
+  </link>
+  <joint name="camera_joint" type="fixed">
+    <parent link="base_link"/>
+    <child link="camera_link"/>
+    <origin xyz="0.15 0 0.1" rpy="0 0 0"/>
+  </joint>
+  <gazebo reference="camera_link">
+    <sensor type="camera" name="camera">
+      <always_on>true</always_on>
       <update_rate>30</update_rate>
       <camera>
@@ -38,9 +123,8 @@
       <plugin name="camera_controller" filename="libgazebo_ros_camera.so">
         <ros>
-          <namespace>/lane_robot</namespace>
           <remapping>image_raw:=/camera/image_raw</remapping>
         </ros>
       </plugin>
     </sensor>
-  </link>
+  </gazebo>
 </robot>
